File: spla-board/spla-board.sch (KiCad schematic (older format))
At the start: 0 parts

Commit message: schematic: Remove SRAM, since I don't have the pins for it anyways.
Other:
- note removed: "100 MHz"
- note removed: "32-bit R/W bus"
Changed lines of the file:
@@
 $Descr A3 16535 11693
 encoding utf-8
-Sheet 1 8
+Sheet 1 7
 Title "SPLA Board - Root"
 Date "2020-03-07"
@@
 F1 "spla-board-power.sch" 50
 $EndSheet
-$Sheet
-S 5500 6500 1500 1000
-U 5E50D3C6
-F0 "SPLA Board - SRAM" 50
-F1 "spla-board-sram.sch" 50
-$EndSheet
 Wire Notes Line width 12 style solid
 	3000 5000 4500 5000
@@
 Wire Notes Line width 12 style solid
 	8100 6500 8100 5500
-Wire Notes Line width 12 style solid
-	7000 5400 6700 5400
-Wire Notes Line width 12 style solid
-	6700 5400 6700 6500
-Text Notes 6650 6200 1    50   ~ 0
-32-bit R/W bus
 Text Notes 6350 5100 0    50   ~ 0
 60 MHz
@@
 Text Notes 8350 6600 0    25   ~ 0
 21.47727 MHz\n3.579545 MHz
-Text Notes 6800 6050 1    50   ~ 0
-100 MHz
 Text Notes 3350 5100 0    50   ~ 0
 480 Mbps / 60MBps

Commit message: schematic: Correct ADC bus width.
Other:
- note added: "24-bit R/G/B bus"
- note removed: "30-bit R/G/B bus"
Changed lines of the file:
@@
 Analog R/G/B
 Text Notes 8900 6450 2    50   ~ 0
-30-bit R/G/B bus
+24-bit R/G/B bus
 Wire Notes Line style solid
 	7500 2700 7800 2700
