File: spla-board/spla-board-fpga.sch (KiCad schematic (older format))
At the start: 35 parts, among them J2 J_JTAG, U1 LFE5U-45F-BG256

Commit message: schematic/pcb: Complete part selection of resistors and capacitors.  Omit filters in analog block for now; adjust PCB to suit.
Parts:
- C13, C31: Digikey (none) -> 490-16477-1-ND; Manufacturer (none) -> Murata Electronics; Manufacturer Id (none) -> GCJ188R71E104KA12D
- C15, C17, C19, C20, C21, C23, C24, C25, C27, C30, C32, C33, C34, C35, C37: Digikey (none) -> 490-6351-1-ND; Manufacturer (none) -> Murata Electronics; Manufacturer Id (none) -> GRM155R71H103KA88J
- R10, R26, R27, R9: Digikey (none) -> RMCF0603JT330RCT-ND; Manufacturer (none) -> Stackpole Electronics Inc; Manufacturer Id (none) -> RMCF0603JT330R
- R13, R14, R16, R28: Digikey (none) -> RMCF0603JT4K70CT-ND; Manufacturer (none) -> Stackpole Electronics Inc; Manufacturer Id (none) -> RMCF0603JT4K70
- R15: Digikey (none) -> RMCF0402FT4K70CT-ND; Manufacturer (none) -> Stackpole Electronics Inc; Manufacturer Id (none) -> RMCF0402FT4K70
Changed lines of the file:
@@
 F 2 "Resistor_SMD:R_0603_1608Metric" H 3400 9750 50  0001 C CNN
 F 3 "~" H 3400 9750 50  0001 C CNN
+F 4 "RMCF0603JT4K70CT-ND" H 3400 9750 50  0001 C CNN "Digikey"
+F 5 "Stackpole Electronics Inc" H 3400 9750 50  0001 C CNN "Manufacturer"
+F 6 "RMCF0603JT4K70" H 3400 9750 50  0001 C CNN "Manufacturer Id"
 	1    3400 9750
 	1    0    0    -1
@@
 F 2 "Resistor_SMD:R_0603_1608Metric" H 3400 10450 50  0001 C CNN
 F 3 "~" H 3400 10450 50  0001 C CNN
+F 4 "RMCF0603JT4K70CT-ND" H 3400 10450 50  0001 C CNN "Digikey"
+F 5 "Stackpole Electronics Inc" H 3400 10450 50  0001 C CNN "Manufacturer"
+F 6 "RMCF0603JT4K70" H 3400 10450 50  0001 C CNN "Manufacturer Id"
 	1    3400 10450
 	1    0    0    -1
@@
 F 2 "Resistor_SMD:R_0603_1608Metric" H 5550 10100 50  0001 C CNN
 F 3 "~" H 5550 10100 50  0001 C CNN
+F 4 "RMCF0603JT330RCT-ND" H 5550 10100 50  0001 C CNN "Digikey"
+F 5 "Stackpole Electronics Inc" H 5550 10100 50  0001 C CNN "Manufacturer"
+F 6 "RMCF0603JT330R" H 5550 10100 50  0001 C CNN "Manufacturer Id"
 	1    5550 10100
 	1    0    0    -1
@@
 F 2 "Resistor_SMD:R_0603_1608Metric" H 5950 10100 50  0001 C CNN
 F 3 "~" H 5950 10100 50  0001 C CNN
+F 4 "RMCF0603JT330RCT-ND" H 5950 10100 50  0001 C CNN "Digikey"
+F 5 "Stackpole Electronics Inc" H 5950 10100 50  0001 C CNN "Manufacturer"
+F 6 "RMCF0603JT330R" H 5950 10100 50  0001 C CNN "Manufacturer Id"
 	1    5950 10100
 	1    0    0    -1
@@
 F 2 "Resistor_SMD:R_0603_1608Metric" H 4750 10100 50  0001 C CNN
 F 3 "~" H 4750 10100 50  0001 C CNN
+F 4 "RMCF0603JT330RCT-ND" H 4750 10100 50  0001 C CNN "Digikey"
+F 5 "Stackpole Electronics Inc" H 4750 10100 50  0001 C CNN "Manufacturer"
+F 6 "RMCF0603JT330R" H 4750 10100 50  0001 C CNN "Manufacturer Id"
 	1    4750 10100
 	1    0    0    -1
@@
 F 2 "Resistor_SMD:R_0603_1608Metric" H 5150 10100 50  0001 C CNN
 F 3 "~" H 5150 10100 50  0001 C CNN
+F 4 "RMCF0603JT330RCT-ND" H 5150 10100 50  0001 C CNN "Digikey"
+F 5 "Stackpole Electronics Inc" H 5150 10100 50  0001 C CNN "Manufacturer"
+F 6 "RMCF0603JT330R" H 5150 10100 50  0001 C CNN "Manufacturer Id"
 	1    5150 10100
 	1    0    0    -1
@@
 F 2 "Resistor_SMD:R_0402_1005Metric" H 4000 6800 50  0001 C CNN
 F 3 "~" H 4000 6800 50  0001 C CNN
+F 4 "RMCF0402FT4K70CT-ND" H 4000 6800 50  0001 C CNN "Digikey"
+F 5 "Stackpole Electronics Inc" H 4000 6800 50  0001 C CNN "Manufacturer"
+F 6 "RMCF0402FT4K70" H 4000 6800 50  0001 C CNN "Manufacturer Id"
 	1    4000 6800
 	1    0    0    -1
@@
 F 2 "Resistor_SMD:R_0603_1608Metric" H 4500 8500 50  0001 C CNN
 F 3 "~" H 4500 8500 50  0001 C CNN
+F 4 "RMCF0603JT4K70CT-ND" H 4500 8500 50  0001 C CNN "Digikey"
+F 5 "Stackpole Electronics Inc" H 4500 8500 50  0001 C CNN "Manufacturer"
+F 6 "RMCF0603JT4K70" H 4500 8500 50  0001 C CNN "Manufacturer Id"
 	1    4500 8500
 	1    0    0    -1
@@
 F 2 "Resistor_SMD:R_0603_1608Metric" H 5200 8500 50  0001 C CNN
 F 3 "~" H 5200 8500 50  0001 C CNN
+F 4 "RMCF0603JT4K70CT-ND" H 5200 8500 50  0001 C CNN "Digikey"
+F 5 "Stackpole Electronics Inc" H 5200 8500 50  0001 C CNN "Manufacturer"
+F 6 "RMCF0603JT4K70" H 5200 8500 50  0001 C CNN "Manufacturer Id"
 	1    5200 8500
 	1    0    0    -1
@@
 F 2 "Capacitor_SMD:C_0603_1608Metric" H 7750 6700 50  0001 C CNN
 F 3 "~" H 7750 6700 50  0001 C CNN
+F 4 "490-16477-1-ND" H 7750 6700 50  0001 C CNN "Digikey"
+F 5 "Murata Electronics" H 7750 6700 50  0001 C CNN "Manufacturer"
+F 6 "GCJ188R71E104KA12D" H 7750 6700 50  0001 C CNN "Manufacturer Id"
 	1    7750 6700
 	1    0    0    -1
@@
 F 2 "Capacitor_SMD:C_0402_1005Metric" H 7750 7800 50  0001 C CNN
 F 3 "~" H 7750 7800 50  0001 C CNN
+F 4 "490-6351-1-ND" H 7750 7800 50  0001 C CNN "Digikey"
+F 5 "Murata Electronics" H 7750 7800 50  0001 C CNN "Manufacturer"
+F 6 "GRM155R71H103KA88J" H 7750 7800 50  0001 C CNN "Manufacturer Id"
 	1    7750 7800
 	1    0    0    -1
@@
 F 2 "Capacitor_SMD:C_0402_1005Metric" H 8200 7800 50  0001 C CNN
 F 3 "~" H 8200 7800 50  0001 C CNN
+F 4 "490-6351-1-ND" H 8200 7800 50  0001 C CNN "Digikey"
+F 5 "Murata Electronics" H 8200 7800 50  0001 C CNN "Manufacturer"
+F 6 "GRM155R71H103KA88J" H 8200 7800 50  0001 C CNN "Manufacturer Id"
 	1    8200 7800
 	1    0    0    -1
@@
 F 2 "Capacitor_SMD:C_0402_1005Metric" H 8650 7800 50  0001 C CNN
 F 3 "~" H 8650 7800 50  0001 C CNN
+F 4 "490-6351-1-ND" H 8650 7800 50  0001 C CNN "Digikey"
+F 5 "Murata Electronics" H 8650 7800 50  0001 C CNN "Manufacturer"
+F 6 "GRM155R71H103KA88J" H 8650 7800 50  0001 C CNN "Manufacturer Id"
 	1    8650 7800
 	1    0    0    -1
@@
 F 2 "Capacitor_SMD:C_0402_1005Metric" H 8200 6700 50  0001 C CNN
 F 3 "~" H 8200 6700 50  0001 C CNN
+F 4 "490-6351-1-ND" H 8200 6700 50  0001 C CNN "Digikey"
+F 5 "Murata Electronics" H 8200 6700 50  0001 C CNN "Manufacturer"
+F 6 "GRM155R71H103KA88J" H 8200 6700 50  0001 C CNN "Manufacturer Id"
 	1    8200 6700
 	1    0    0    -1
@@
 F 2 "Capacitor_SMD:C_0402_1005Metric" H 8650 6700 50  0001 C CNN
 F 3 "~" H 8650 6700 50  0001 C CNN
+F 4 "490-6351-1-ND" H 8650 6700 50  0001 C CNN "Digikey"
+F 5 "Murata Electronics" H 8650 6700 50  0001 C CNN "Manufacturer"
+F 6 "GRM155R71H103KA88J" H 8650 6700 50  0001 C CNN "Manufacturer Id"
 	1    8650 6700
 	1    0    0    -1
@@
 F 2 "Capacitor_SMD:C_0402_1005Metric" H 9100 6700 50  0001 C CNN
 F 3 "~" H 9100 6700 50  0001 C CNN
+F 4 "490-6351-1-ND" H 9100 6700 50  0001 C CNN "Digikey"
+F 5 "Murata Electronics" H 9100 6700 50  0001 C CNN "Manufacturer"
+F 6 "GRM155R71H103KA88J" H 9100 6700 50  0001 C CNN "Manufacturer Id"
 	1    9100 6700
 	1    0    0    -1
@@
 F 2 "Capacitor_SMD:C_0402_1005Metric" H 13150 6700 50  0001 C CNN
 F 3 "~" H 13150 6700 50  0001 C CNN
+F 4 "490-6351-1-ND" H 13150 6700 50  0001 C CNN "Digikey"
+F 5 "Murata Electronics" H 13150 6700 50  0001 C CNN "Manufacturer"
+F 6 "GRM155R71H103KA88J" H 13150 6700 50  0001 C CNN "Manufacturer Id"
 	1    13150 6700
 	1    0    0    -1
@@
 F 2 "Capacitor_SMD:C_0603_1608Metric" H 12700 6700 50  0001 C CNN
 F 3 "~" H 12700 6700 50  0001 C CNN
+F 4 "490-16477-1-ND" H 12700 6700 50  0001 C CNN "Digikey"
+F 5 "Murata Electronics" H 12700 6700 50  0001 C CNN "Manufacturer"
+F 6 "GCJ188R71E104KA12D" H 12700 6700 50  0001 C CNN "Manufacturer Id"
 	1    12700 6700
 	1    0    0    -1
@@
 F 2 "Capacitor_SMD:C_0402_1005Metric" H 13600 6700 50  0001 C CNN
 F 3 "~" H 13600 6700 50  0001 C CNN
+F 4 "490-6351-1-ND" H 13600 6700 50  0001 C CNN "Digikey"
+F 5 "Murata Electronics" H 13600 6700 50  0001 C CNN "Manufacturer"
+F 6 "GRM155R71H103KA88J" H 13600 6700 50  0001 C CNN "Manufacturer Id"
 	1    13600 6700
 	1    0    0    -1
@@
 F 2 "Capacitor_SMD:C_0402_1005Metric" H 10450 6700 50  0001 C CNN
 F 3 "~" H 10450 6700 50  0001 C CNN
+F 4 "490-6351-1-ND" H 10450 6700 50  0001 C CNN "Digikey"
+F 5 "Murata Electronics" H 10450 6700 50  0001 C CNN "Manufacturer"
+F 6 "GRM155R71H103KA88J" H 10450 6700 50  0001 C CNN "Manufacturer Id"
 	1    10450 6700
 	1    0    0    -1
@@
 F 2 "Capacitor_SMD:C_0402_1005Metric" H 10000 6700 50  0001 C CNN
 F 3 "~" H 10000 6700 50  0001 C CNN
+F 4 "490-6351-1-ND" H 10000 6700 50  0001 C CNN "Digikey"
+F 5 "Murata Electronics" H 10000 6700 50  0001 C CNN "Manufacturer"
+F 6 "GRM155R71H103KA88J" H 10000 6700 50  0001 C CNN "Manufacturer Id"
 	1    10000 6700
 	1    0    0    -1
@@
 F 2 "Capacitor_SMD:C_0402_1005Metric" H 9550 6700 50  0001 C CNN
 F 3 "~" H 9550 6700 50  0001 C CNN
+F 4 "490-6351-1-ND" H 9550 6700 50  0001 C CNN "Digikey"
+F 5 "Murata Electronics" H 9550 6700 50  0001 C CNN "Manufacturer"
+F 6 "GRM155R71H103KA88J" H 9550 6700 50  0001 C CNN "Manufacturer Id"
 	1    9550 6700
 	1    0    0    -1
@@
 F 2 "Capacitor_SMD:C_0402_1005Metric" H 9100 7800 50  0001 C CNN
 F 3 "~" H 9100 7800 50  0001 C CNN
+F 4 "490-6351-1-ND" H 9100 7800 50  0001 C CNN "Digikey"
+F 5 "Murata Electronics" H 9100 7800 50  0001 C CNN "Manufacturer"
+F 6 "GRM155R71H103KA88J" H 9100 7800 50  0001 C CNN "Manufacturer Id"
 	1    9100 7800
 	1    0    0    -1
@@
 F 2 "Capacitor_SMD:C_0402_1005Metric" H 9550 7800 50  0001 C CNN
 F 3 "~" H 9550 7800 50  0001 C CNN
+F 4 "490-6351-1-ND" H 9550 7800 50  0001 C CNN "Digikey"
+F 5 "Murata Electronics" H 9550 7800 50  0001 C CNN "Manufacturer"
+F 6 "GRM155R71H103KA88J" H 9550 7800 50  0001 C CNN "Manufacturer Id"
 	1    9550 7800
 	1    0    0    -1
@@
 F 2 "Capacitor_SMD:C_0402_1005Metric" H 10000 7800 50  0001 C CNN
 F 3 "~" H 10000 7800 50  0001 C CNN
+F 4 "490-6351-1-ND" H 10000 7800 50  0001 C CNN "Digikey"
+F 5 "Murata Electronics" H 10000 7800 50  0001 C CNN "Manufacturer"
+F 6 "GRM155R71H103KA88J" H 10000 7800 50  0001 C CNN "Manufacturer Id"
 	1    10000 7800
 	1    0    0    -1
@@
 F 2 "Capacitor_SMD:C_0402_1005Metric" H 10450 7800 50  0001 C CNN
 F 3 "~" H 10450 7800 50  0001 C CNN
+F 4 "490-6351-1-ND" H 10450 7800 50  0001 C CNN "Digikey"
+F 5 "Murata Electronics" H 10450 7800 50  0001 C CNN "Manufacturer"
+F 6 "GRM155R71H103KA88J" H 10450 7800 50  0001 C CNN "Manufacturer Id"
 	1    10450 7800
 	1    0    0    -1
