File: spla-board/spla-board-level-shifters.sch (KiCad schematic (older format))
At the start: 22 parts, among them J3 J_BODGE, J6 J_SAMPLE, U15 74LVC8T245, U16 74LVC8T245, U17 74LVC8T245, U20 74LVC8T245, U22 74LVC8T245, U23 74LVC8T245, U24 74LVC8T245, U25 74LVC8T245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

Commit message: schematic/pcb: Complete part selection of resistors and capacitors.  Omit filters in analog block for now; adjust PCB to suit.
Parts:
- R25: Digikey (none) -> 2019-RK73Z1JTTDCT-ND; Manufacturer (none) -> KOA Speer Electronics Inc.; Manufacturer Id (none) -> RK73Z1JTTD
- R29, R30: Digikey (none) -> RMCF0603JT10K0CT-ND; Manufacturer (none) -> Stackpole Electronics Inc; Manufacturer Id (none) -> RMCF0603JT10K0
Changed lines of the file:
@@
 F 2 "Resistor_SMD:R_0603_1608Metric" H 1250 4200 50  0001 C CNN
 F 3 "~" H 1250 4200 50  0001 C CNN
+F 4 "2019-RK73Z1JTTDCT-ND" H 1250 4200 50  0001 C CNN "Digikey"
+F 5 "KOA Speer Electronics Inc." H 1250 4200 50  0001 C CNN "Manufacturer"
+F 6 "RK73Z1JTTD" H 1250 4200 50  0001 C CNN "Manufacturer Id"
 	1    1250 4200
 	1    0    0    -1
@@
 F 2 "Resistor_SMD:R_0603_1608Metric" H 1250 2150 50  0001 C CNN
 F 3 "~" H 1250 2150 50  0001 C CNN
+F 4 "RMCF0603JT10K0CT-ND" H 1250 2150 50  0001 C CNN "Digikey"
+F 5 "Stackpole Electronics Inc" H 1250 2150 50  0001 C CNN "Manufacturer"
+F 6 "RMCF0603JT10K0" H 1250 2150 50  0001 C CNN "Manufacturer Id"
 	1    1250 2150
 	1    0    0    -1
@@
 F 2 "Resistor_SMD:R_0603_1608Metric" H 1550 2150 50  0001 C CNN
 F 3 "~" H 1550 2150 50  0001 C CNN
+F 4 "RMCF0603JT10K0CT-ND" H 1550 2150 50  0001 C CNN "Digikey"
+F 5 "Stackpole Electronics Inc" H 1550 2150 50  0001 C CNN "Manufacturer"
+F 6 "RMCF0603JT10K0" H 1550 2150 50  0001 C CNN "Manufacturer Id"
 	1    1550 2150
 	1    0    0    -1
