File: spla-board/spla-board-ppu.sch (KiCad schematic (older format))
At the start: 22 parts, among them J15 J_DPULL, J5 J_PPURESET, U10 SNES_PPU1, U11 SNES_PPU2, U12 VRAM, U13 VRAM

Commit message: schematic/pcb: Complete part selection of resistors and capacitors.  Omit filters in analog block for now; adjust PCB to suit.
Parts:
- C10, C12, C8, C9: Digikey (none) -> 490-16477-1-ND; Manufacturer (none) -> Murata Electronics; Manufacturer Id (none) -> GCJ188R71E104KA12D
- C11: Digikey (none) -> 490-17769-1-ND; Manufacturer (none) -> Murata Electronics; Manufacturer Id (none) -> GCM1885C2A560JA16D
- R11: Digikey (none) -> RMCF0603JT100RCT-ND; Manufacturer (none) -> Stackpole Electronics Inc; Manufacturer Id (none) -> RMCF0603JT100R
- R17, R18, R19, R20, R21, R22, R23, R24: Digikey (none) -> RMCF0603JT10K0CT-ND; Manufacturer (none) -> Stackpole Electronics Inc; Manufacturer Id (none) -> RMCF0603JT10K0
Changed lines of the file:
@@
 F 2 "Resistor_SMD:R_0603_1608Metric" V 10380 5800 50  0001 C CNN
 F 3 "~" H 10450 5800 50  0001 C CNN
+F 4 "RMCF0603JT100RCT-ND" H 10450 5800 50  0001 C CNN "Digikey"
+F 5 "Stackpole Electronics Inc" H 10450 5800 50  0001 C CNN "Manufacturer"
+F 6 "RMCF0603JT100R" H 10450 5800 50  0001 C CNN "Manufacturer Id"
 	1    10450 5800
 	1    0    0    -1
@@
 F 2 "Capacitor_SMD:C_0603_1608Metric" H 10488 5950 50  0001 C CNN
 F 3 "~" H 10450 6100 50  0001 C CNN
+F 4 "490-17769-1-ND" H 10450 6100 50  0001 C CNN "Digikey"
+F 5 "Murata Electronics" H 10450 6100 50  0001 C CNN "Manufacturer"
+F 6 "GCM1885C2A560JA16D" H 10450 6100 50  0001 C CNN "Manufacturer Id"
 	1    10450 6100
 	1    0    0    -1
@@
 F 2 "Capacitor_SMD:C_0603_1608Metric" H 6700 3100 50  0001 C CNN
 F 3 "~" H 6700 3100 50  0001 C CNN
+F 4 "490-16477-1-ND" H 6700 3100 50  0001 C CNN "Digikey"
+F 5 "Murata Electronics" H 6700 3100 50  0001 C CNN "Manufacturer"
+F 6 "GCJ188R71E104KA12D" H 6700 3100 50  0001 C CNN "Manufacturer Id"
 	1    6700 3100
 	1    0    0    -1
@@
 F 2 "Capacitor_SMD:C_0603_1608Metric" H 13000 3100 50  0001 C CNN
 F 3 "~" H 13000 3100 50  0001 C CNN
+F 4 "490-16477-1-ND" H 13000 3100 50  0001 C CNN "Digikey"
+F 5 "Murata Electronics" H 13000 3100 50  0001 C CNN "Manufacturer"
+F 6 "GCJ188R71E104KA12D" H 13000 3100 50  0001 C CNN "Manufacturer Id"
 	1    13000 3100
 	1    0    0    -1
@@
 F 2 "Capacitor_SMD:C_0603_1608Metric" H 9400 3200 50  0001 C CNN
 F 3 "~" H 9400 3200 50  0001 C CNN
+F 4 "490-16477-1-ND" H 9400 3200 50  0001 C CNN "Digikey"
+F 5 "Murata Electronics" H 9400 3200 50  0001 C CNN "Manufacturer"
+F 6 "GCJ188R71E104KA12D" H 9400 3200 50  0001 C CNN "Manufacturer Id"
 	1    9400 3200
 	1    0    0    -1
@@
 F 2 "Capacitor_SMD:C_0603_1608Metric" H 9400 5500 50  0001 C CNN
 F 3 "~" H 9400 5500 50  0001 C CNN
+F 4 "490-16477-1-ND" H 9400 5500 50  0001 C CNN "Digikey"
+F 5 "Murata Electronics" H 9400 5500 50  0001 C CNN "Manufacturer"
+F 6 "GCJ188R71E104KA12D" H 9400 5500 50  0001 C CNN "Manufacturer Id"
 	1    9400 5500
 	1    0    0    -1
@@
 F 2 "Resistor_SMD:R_0603_1608Metric" H 3800 8750 50  0001 C CNN
 F 3 "~" H 3800 8750 50  0001 C CNN
+F 4 "RMCF0603JT10K0CT-ND" H 3800 8750 50  0001 C CNN "Digikey"
+F 5 "Stackpole Electronics Inc" H 3800 8750 50  0001 C CNN "Manufacturer"
+F 6 "RMCF0603JT10K0" H 3800 8750 50  0001 C CNN "Manufacturer Id"
 	1    3800 8750
 	1    0    0    -1
@@
 F 2 "Resistor_SMD:R_0603_1608Metric" H 3550 8750 50  0001 C CNN
 F 3 "~" H 3550 8750 50  0001 C CNN
+F 4 "RMCF0603JT10K0CT-ND" H 3550 8750 50  0001 C CNN "Digikey"
+F 5 "Stackpole Electronics Inc" H 3550 8750 50  0001 C CNN "Manufacturer"
+F 6 "RMCF0603JT10K0" H 3550 8750 50  0001 C CNN "Manufacturer Id"
 	1    3550 8750
 	1    0    0    -1
@@
 F 2 "Resistor_SMD:R_0603_1608Metric" H 3300 8750 50  0001 C CNN
 F 3 "~" H 3300 8750 50  0001 C CNN
+F 4 "RMCF0603JT10K0CT-ND" H 3300 8750 50  0001 C CNN "Digikey"
+F 5 "Stackpole Electronics Inc" H 3300 8750 50  0001 C CNN "Manufacturer"
+F 6 "RMCF0603JT10K0" H 3300 8750 50  0001 C CNN "Manufacturer Id"
 	1    3300 8750
 	1    0    0    -1
@@
 F 2 "Resistor_SMD:R_0603_1608Metric" H 3050 8750 50  0001 C CNN
 F 3 "~" H 3050 8750 50  0001 C CNN
+F 4 "RMCF0603JT10K0CT-ND" H 3050 8750 50  0001 C CNN "Digikey"
+F 5 "Stackpole Electronics Inc" H 3050 8750 50  0001 C CNN "Manufacturer"
+F 6 "RMCF0603JT10K0" H 3050 8750 50  0001 C CNN "Manufacturer Id"
 	1    3050 8750
 	1    0    0    -1
@@
 F 2 "Resistor_SMD:R_0603_1608Metric" H 2800 8750 50  0001 C CNN
 F 3 "~" H 2800 8750 50  0001 C CNN
+F 4 "RMCF0603JT10K0CT-ND" H 2800 8750 50  0001 C CNN "Digikey"
+F 5 "Stackpole Electronics Inc" H 2800 8750 50  0001 C CNN "Manufacturer"
+F 6 "RMCF0603JT10K0" H 2800 8750 50  0001 C CNN "Manufacturer Id"
 	1    2800 8750
 	1    0    0    -1
@@
 F 2 "Resistor_SMD:R_0603_1608Metric" H 2550 8750 50  0001 C CNN
 F 3 "~" H 2550 8750 50  0001 C CNN
+F 4 "RMCF0603JT10K0CT-ND" H 2550 8750 50  0001 C CNN "Digikey"
+F 5 "Stackpole Electronics Inc" H 2550 8750 50  0001 C CNN "Manufacturer"
+F 6 "RMCF0603JT10K0" H 2550 8750 50  0001 C CNN "Manufacturer Id"
 	1    2550 8750
 	1    0    0    -1
@@
 F 2 "Resistor_SMD:R_0603_1608Metric" H 2300 8750 50  0001 C CNN
 F 3 "~" H 2300 8750 50  0001 C CNN
+F 4 "RMCF0603JT10K0CT-ND" H 2300 8750 50  0001 C CNN "Digikey"
+F 5 "Stackpole Electronics Inc" H 2300 8750 50  0001 C CNN "Manufacturer"
+F 6 "RMCF0603JT10K0" H 2300 8750 50  0001 C CNN "Manufacturer Id"
 	1    2300 8750
 	1    0    0    -1
@@
 F 2 "Resistor_SMD:R_0603_1608Metric" H 2050 8750 50  0001 C CNN
 F 3 "~" H 2050 8750 50  0001 C CNN
+F 4 "RMCF0603JT10K0CT-ND" H 2050 8750 50  0001 C CNN "Digikey"
+F 5 "Stackpole Electronics Inc" H 2050 8750 50  0001 C CNN "Manufacturer"
+F 6 "RMCF0603JT10K0" H 2050 8750 50  0001 C CNN "Manufacturer Id"
 	1    2050 8750
 	1    0    0    -1
@@
 	1    0    0    -1
 $EndComp
+Wire Wire Line
+	11150 2600 11600 2600
+Text GLabel 11600 2600 2    50   Input ~ 0
+TAP_PPU2_~RESET~
 Wire Bus Line
 	10200 2700 10200 6050
@@
 	3350 2700 3350 6550
 Wire Bus Line
+	4550 2600 4550 5150
+Wire Bus Line
+	10850 2600 10850 5450
+Wire Bus Line
 	6800 7050 6800 9400
-Wire Bus Line
-	13350 6150 13350 9400
-Wire Bus Line
-	10000 4350 10000 9400
 Wire Bus Line
 	11100 6950 11100 9500
@@
 	4550 6950 4550 9500
 Wire Bus Line
-	10850 2600 10850 5450
+	6800 3400 6800 6650
 Wire Bus Line
 	8200 3400 8200 7150
 Wire Bus Line
-	6800 3400 6800 6650
+	13350 6150 13350 9400
 Wire Bus Line
-	4550 2600 4550 5150
-Wire Wire Line
-	11150 2600 11600 2600
-Text GLabel 11600 2600 2    50   Input ~ 0
-TAP_PPU2_~RESET~
+	10000 4350 10000 9400
 $EndSCHEMATC
