File: spla-board/spla-board-usb.sch (KiCad schematic (older format))
At the start: 27 parts, among them J1 USB_B_Micro, U2 FT2232H, U3 93LC66B, X1 FT5HNBPK12.0-T1

Commit message: schematic/pcb: Add 12mhz clock test point; renumber test points.
Parts:
- added TP6: TP_12MHZ, TestPoint:TestPoint_Pad_D1.0mm, symbol Connector:TestPoint
- renumbered TP10 to TP5
Connections:
- net CLK_12MHZ: now also TP6.1
Other:
- moved on the sheet: C14, X1
Changed lines of the file:
@@
 L power:GND #PWR0105
 U 1 1 5E58FEB5
-P 6350 8000
-F 0 "#PWR0105" H 6350 7750 50  0001 C CNN
-F 1 "GND" H 6355 7827 50  0000 C CNN
-F 2 "" H 6350 8000 50  0001 C CNN
-F 3 "" H 6350 8000 50  0001 C CNN
-	1    6350 8000
+P 6150 8000
+F 0 "#PWR0105" H 6150 7750 50  0001 C CNN
+F 1 "GND" H 6155 7827 50  0000 C CNN
+F 2 "" H 6150 8000 50  0001 C CNN
+F 3 "" H 6150 8000 50  0001 C CNN
+	1    6150 8000
 	1    0    0    -1
 $EndComp
@@
 L power:+3V3 #PWR0109
 U 1 1 5E649611
-P 6350 7350
-F 0 "#PWR0109" H 6350 7200 50  0001 C CNN
-F 1 "+3V3" H 6365 7523 50  0000 C CNN
-F 2 "" H 6350 7350 50  0001 C CNN
-F 3 "" H 6350 7350 50  0001 C CNN
-	1    6350 7350
+P 6150 7350
+F 0 "#PWR0109" H 6150 7200 50  0001 C CNN
+F 1 "+3V3" H 6165 7523 50  0000 C CNN
+F 2 "" H 6150 7350 50  0001 C CNN
+F 3 "" H 6150 7350 50  0001 C CNN
+	1    6150 7350
 	1    0    0    -1
 $EndComp
@@
 L SPLA:FT5HNBPK12.0-T1 X1
 U 1 1 5FDCFC82
-P 7150 7800
+P 6950 7800
 AR Path="/5FDCFC82" Ref="X1"  Part="1"
 AR Path="/5E4F712F/5FDCFC82" Ref="X1"  Part="1"
-F 0 "X1" H 6850 8050 50  0000 L CNN
-F 1 "FT5HNBPK12.0-T1" H 7150 7550 50  0000 C CNN
-F 2 "Crystal:Crystal_SMD_5032-4Pin_5.0x3.2mm" H 7200 7300 50  0001 C CNN
-F 3 "" H 7580 7490 50  0001 C CNN
-F 4 "631-1068-1-ND" H 7150 7800 50  0001 C CNN "Digikey"
-F 5 "FT5HNBPK12.0-T1" H 7150 7800 50  0001 C CNN "Manufacturer Id"
-F 6 "Fox Electronics" H 7150 7800 50  0001 C CNN "Manufacturer"
-	1    7150 7800
-	1    0    0    -1
-$EndComp
-Wire Wire Line
-	6750 7900 6350 7900
-Wire Wire Line
-	7550 7700 7550 7450
-Connection ~ 6350 7900
+F 0 "X1" H 6650 8050 50  0000 L CNN
+F 1 "FT5HNBPK12.0-T1" H 6950 7550 50  0000 C CNN
+F 2 "Crystal:Crystal_SMD_5032-4Pin_5.0x3.2mm" H 7000 7300 50  0001 C CNN
+F 3 "" H 7380 7490 50  0001 C CNN
+F 4 "631-1068-1-ND" H 6950 7800 50  0001 C CNN "Digikey"
+F 5 "FT5HNBPK12.0-T1" H 6950 7800 50  0001 C CNN "Manufacturer Id"
+F 6 "Fox Electronics" H 6950 7800 50  0001 C CNN "Manufacturer"
+	1    6950 7800
+	1    0    0    -1
+$EndComp
+Wire Wire Line
+	6550 7900 6150 7900
+Wire Wire Line
+	7350 7700 7350 7450
+Connection ~ 6150 7900
 NoConn ~ 11150 5050
 Text GLabel 11150 6050 2    39   BiDi ~ 0
@@
 	3100 4750 8750 4750
 Wire Wire Line
-	6350 7450 6350 7600
-Wire Wire Line
-	6350 7800 6350 7900
+	6150 7450 6150 7600
+Wire Wire Line
+	6150 7800 6150 7900
 Text GLabel 11150 7350 2    39   Output ~ 0
 USB_~PWREN~
@@
 $EndComp
 Wire Wire Line
-	6350 7450 7550 7450
-NoConn ~ 6750 7700
-Connection ~ 6350 7450
-Wire Wire Line
-	6350 7450 6350 7350
-Wire Wire Line
-	6350 7900 6350 8000
+	6150 7450 7350 7450
+NoConn ~ 6550 7700
+Connection ~ 6150 7450
+Wire Wire Line
+	6150 7450 6150 7350
+Wire Wire Line
+	6150 7900 6150 8000
 $Comp
 L SPLA:BomExtra BOM1
@@
 L Device:C_Small C14
 U 1 1 5E53DEA7
-P 6350 7700
-F 0 "C14" H 6465 7746 50  0000 L CNN
-F 1 "0.1uF" H 6465 7655 50  0000 L CNN
-F 2 "Capacitor_SMD:C_0603_1608Metric" H 6388 7550 50  0001 C CNN
-F 3 "~" H 6350 7700 50  0001 C CNN
-F 4 "490-16477-1-ND" H 6350 7700 50  0001 C CNN "Digikey"
-F 5 "Murata Electronics" H 6350 7700 50  0001 C CNN "Manufacturer"
-F 6 "GCJ188R71E104KA12D" H 6350 7700 50  0001 C CNN "Manufacturer Id"
-	1    6350 7700
+P 6150 7700
+F 0 "C14" H 6265 7746 50  0000 L CNN
+F 1 "0.1uF" H 6265 7655 50  0000 L CNN
+F 2 "Capacitor_SMD:C_0603_1608Metric" H 6188 7550 50  0001 C CNN
+F 3 "~" H 6150 7700 50  0001 C CNN
+F 4 "490-16477-1-ND" H 6150 7700 50  0001 C CNN "Digikey"
+F 5 "Murata Electronics" H 6150 7700 50  0001 C CNN "Manufacturer"
+F 6 "GCJ188R71E104KA12D" H 6150 7700 50  0001 C CNN "Manufacturer Id"
+	1    6150 7700
 	1    0    0    -1
 $EndComp
@@
 NoConn ~ 3650 5050
 $Comp
-L Connector:TestPoint TP10
+L Connector:TestPoint TP5
 U 1 1 5F33FE5B
 P 7700 3800
-F 0 "TP10" H 7758 3918 50  0000 L CNN
+F 0 "TP5" H 7758 3918 50  0000 L CNN
 F 1 "TP_1V8" H 7758 3827 50  0000 L CNN
 F 2 "TestPoint:TestPoint_Pad_D1.0mm" H 7900 3800 50  0001 C CNN
@@
 Wire Wire Line
 	8100 8300 8300 8300
-Connection ~ 8100 7900
-Wire Wire Line
-	8100 7900 8100 8300
 Wire Wire Line
 	8100 6850 8750 6850
-Wire Wire Line
-	8100 7900 8100 6850
-Wire Wire Line
-	7550 7900 8100 7900
 $Comp
 L Device:R R3
@@
 	1    0    0    -1
 $EndComp
+$Comp
+L Connector:TestPoint TP6
+U 1 1 5F3A03C0
+P 7600 7800
+F 0 "TP6" H 7658 7918 50  0000 L CNN
+F 1 "TP_12MHZ" H 7658 7827 50  0000 L CNN
+F 2 "TestPoint:TestPoint_Pad_D1.0mm" H 7800 7800 50  0001 C CNN
+F 3 "~" H 7800 7800 50  0001 C CNN
+F 4 "N/A" H 7600 7800 50  0001 C CNN "Digikey"
+F 5 "N/A" H 7600 7800 50  0001 C CNN "Manufacturer"
+F 6 "N/A" H 7600 7800 50  0001 C CNN "Manufacturer Id"
+	1    7600 7800
+	1    0    0    -1
+$EndComp
+Wire Wire Line
+	8100 6850 8100 7900
+Wire Wire Line
+	7350 7900 7600 7900
+Connection ~ 8100 7900
+Wire Wire Line
+	8100 7900 8100 8300
+Wire Wire Line
+	7600 7900 7600 7800
+Connection ~ 7600 7900
+Wire Wire Line
+	7600 7900 8100 7900
 $EndSCHEMATC

Commit message: schematic/pcb: Renumber connectors (J*).
Parts:
- renumbered J1 to J3
Changed lines of the file:
@@
 Decoupling Capacitors\n
 $Comp
-L Connector:USB_B_Micro J1
+L Connector:USB_B_Micro J3
 U 1 1 5E4AA2D6
 P 2800 4850
-F 0 "J1" H 2857 5317 50  0000 C CNN
+F 0 "J3" H 2857 5317 50  0000 C CNN
 F 1 "USB_B_Micro" H 2857 5226 50  0000 C CNN
 F 2 "Connector_USB:USB_Micro-B_Wuerth_629105150521" H 2950 4800 50  0001 C CNN

Commit message: schematic/pcb: Seperate PPU2 AVCC; add more PPU decoupling.
Parts:
- renumbered R73 to R75
Changed lines of the file:
@@
 	11900 5250 11900 5500
 $Comp
-L Device:R R73
+L Device:R R75
 U 1 1 5F36220C
 P 8500 3600
-F 0 "R73" H 8570 3646 50  0000 L CNN
+F 0 "R75" H 8570 3646 50  0000 L CNN
 F 1 "0" H 8570 3555 50  0000 L CNN
 F 2 "Resistor_SMD:R_0603_1608Metric" V 8430 3600 50  0001 C CNN

Commit message: schematic: Swap USB cable for a better (longer) one.
Parts:
- BOM1: Digikey AE11229-ND -> Q966-ND; Manufacturer Assmann WSW Components -> Qualtek; Manufacturer Id AK67421-0.3-VM -> 3025030-03
Changed lines of the file:
@@
 F 2 "SPLA:BoM" H 1600 4850 50  0001 C CNN
 F 3 "" H 1600 4850 50  0001 C CNN
-F 4 "AE11229-ND" H 1600 4850 50  0001 C CNN "Digikey"
-F 5 "AK67421-0.3-VM" H 1600 4850 50  0001 C CNN "Manufacturer Id"
-F 6 "Assmann WSW Components" H 1600 4850 50  0001 C CNN "Manufacturer"
+F 4 "Q966-ND" H 1600 4850 50  0001 C CNN "Digikey"
+F 5 "3025030-03" H 1600 4850 50  0001 C CNN "Manufacturer Id"
+F 6 "Qualtek" H 1600 4850 50  0001 C CNN "Manufacturer"
 	1    1600 4850
 	1    0    0    -1
